File: SubCircuitV3/SubCircuitV3.kicad_pcb (KiCad board)
At the start: 2 copper layers, 121.4 x 121.2 mm, 51 parts, among them J1 JTAG, J10 ESC_POWER, J11 ESC_POWER, J12 ESC_POWER, J13 ESC_POWER, J14 FEMALE XT-60, J15 ESC PWM, J16 5S, J17 Water Sensor Input, J18 3S OUT, J19 2S OUT, J2 ESC PWM, J20 SWITCH, J3 ESC PWM, J4 ESC PWM, J5 ESC PWM, J6 ESC PWM, J7 3S, J8 ESC_POWER, J9 ESC_POWER, K1 G5Q-1A, Q1 NMOS, Q2 NMOS, Q3 NMOS, Q4 NMOS, Q5 NMOS, Q6 NMOS

Commit message: Version 4
Parts:
- added J21: U3V16F15, Connector_PinHeader_2.54mm:PinHeader_1x03_P2.54mm_Vertical, F.Cu at (152.3, 142.3)
- added J22: CAM OUT, 284932-3:CONN3_284392-3_TEC, F.Cu at (136.1, 141.4)
- C1, C2: footprint Capacitor_WCAP-ATG8_5x11_WRE:CAP_WCAP-ATG8_5x11_WRE -> Capacitor_THT:C_Radial_D8.0mm_H7.0mm_P3.50mm
- F7: footprint Resistor_THT:R_Axial_DIN0411_L9.9mm_D3.6mm_P20.32mm_Horizontal -> Resistor_THT:R_Axial_Power_L25.0mm_W9.0mm_P30.48mm
- moved F7 13.1 mm to (174.6, 48.4)
- moved C1 1.32 mm to (133.3, 32.1)
- moved C2 0.47 mm to (154.8, 32.1)
Routing:
- net GND1: track 685.5 -> 724.5 mm
- net +7.5V: track 75.0 -> 61.7 mm
- net +12V: track 352.7 -> 365.5 mm
- net Net-(J21-Pin_1): track 0.00 -> 8.99 mm
- net /SG: track 431.1 -> 434.9 mm
- net GND2: track 220.3 -> 222.9 mm
- net Net-(J19-Pin_3): track 9.11 -> 11.8 mm
- net Net-(CR1-INPUT): track 36.1 -> 38.1 mm
- net Net-(CR1-OUTPUT): track 111.3 -> 113.1 mm
- net Net-(Q2-S): track 25.8 -> 27.6 mm
- net GNDS: track 101.7 -> 101.1 mm

Commit message: newfuse
Parts:
- F8: value Fuse -> 3544-2; footprint Resistor_THT:R_Axial_DIN0411_L9.9mm_D3.6mm_P20.32mm_Horizontal -> 3544-2:FUSE_3544-2
- moved F8 11.9 mm to (177.0, 142.2)
Routing:
- net Net-(J18-Pin_3): track 6.91 -> 16.7 mm
- net +12V: track 365.5 -> 364.2 mm
Changed lines of the file:
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@@
 			(psa4output no)
 			(plot_black_and_white yes)
-			(plotinvisibletext no)
 			(sketchpadsonfab no)
 			(plotpadnumbers no)
@@
 		(embedded_fonts no)
 	)
-	(footprint "Resistor_THT:R_Axial_DIN0411_L9.9mm_D3.6mm_P20.32mm_Horizontal"
+	(footprint "3544-2:FUSE_3544-2"
 		(layer "F.Cu")
-		(at 165.1 143.256)
-		(descr "Resistor, Axial_DIN0411 series, Axial, Horizontal, pin pitch=20.32mm, 1W, length*diameter=9.9*3.6mm^2")
-		(tags "Resistor Axial_DIN0411 series Axial Horizontal pin pitch 20.32mm 1W length 9.9mm diameter 3.6mm")
+		(at 176.985 142.24)
 		(property "Reference" "F8"
-			(at 10.16 -2.92 0)
+			(at -4.445 -3.556 0)
 			(layer "F.SilkS")
 			(effects
@@
 			)
 		)
-		(property "Value" "Fuse"
-			(at 10.16 2.92 0)
+		(property "Value" "3544-2"
+			(at -0.635 4.445 0)
 			(layer "F.Fab")
 			(effects
@@
 		(property "Datasheet" ""
 			(at 0 0 0)
-			(unlocked yes)
 			(layer "F.Fab")
 			(hide yes)
@@
 			)
 		)
-		(property "Description" "Fuse"
+		(property "Description" ""
 			(at 0 0 0)
-			(unlocked yes)
 			(layer "F.Fab")
 			(hide yes)
@@
 			)
 		)
-		(property ki_fp_filters "*Fuse*")
+		(property "PARTREV" "C"
+			(at 0 0 0)
+			(unlocked yes)
+			(layer "F.Fab")
+			(hide yes)
+			(effects
+				(font
+					(size 1 1)
+					(thickness 0.15)
+				)
+			)
+		)
+		(property "STANDARD" "Manufacturer Recommendations"
+			(at 0 0 0)
+			(unlocked yes)
+			(layer "F.Fab")
+			(hide yes)
+			(effects
+				(font
+					(size 1 1)
+					(thickness 0.15)
+				)
+			)
+		)
+		(property "SNAPEDA_PN" "3544-2"
+			(at 0 0 0)
+			(unlocked yes)
+			(layer "F.Fab")
+			(hide yes)
+			(effects
+				(font
+					(size 1 1)
+					(thickness 0.15)
+				)
+			)
+		)
+		(property "MAXIMUM_PACKAGE_HEIGHT" "9.02mm"
+			(at 0 0 0)
+			(unlocked yes)
+			(layer "F.Fab")
+			(hide yes)
+			(effects
+				(font
+					(size 1 1)
+					(thickness 0.15)
+				)
+			)
+		)
+		(property "MANUFACTURER" "Keystone"
+			(at 0 0 0)
+			(unlocked yes)
+			(layer "F.Fab")
+			(hide yes)
+			(effects
+				(font
+					(size 1 1)
+					(thickness 0.15)
+				)
+			)
+		)
 		(sheetname "/")
 		(sheetfile "SubCircuitV3.kicad_sch")
 		(attr through_hole)
 		(fp_line
-			(start 1.44 0)
-			(end 5.09 0)
+			(start -7.34 -2.375)
+			(end -7.34 -1)
 			(stroke
-				(width 0.12)
+				(width 0.127)
 				(type solid)
 			)
@@
 		)
 		(fp_line
-			(start 5.09 -1.92)
-			(end 5.09 1.92)
+			(start -7.34 -2.375)
+			(end 7.34 -2.375)
 			(stroke
-				(width 0.12)
+				(width 0.127)
 				(type solid)
 			)
@@
 		)
 		(fp_line
-			(start 5.09 1.92)
-			(end 15.23 1.92)
+			(start -7.34 1)
+			(end -7.34 2.375)
 			(stroke
-				(width 0.12)
+				(width 0.127)
 				(type solid)
 			)
@@
 		)
 		(fp_line
-			(start 15.23 -1.92)
-			(end 5.09 -1.92)
+			(start 7.34 -2.375)
+			(end 7.34 -1)
 			(stroke
-				(width 0.12)
+				(width 0.127)
 				(type solid)
 			)
@@
 		)
 		(fp_line
-			(start 15.23 1.92)
-			(end 15.23 -1.92)
+			(start 7.34 1)
+			(end 7.34 2.375)
 			(stroke
-				(width 0.12)
+				(width 0.127)
 				(type solid)
 			)
@@
 		)
 		(fp_line
-			(start 18.88 0)
-			(end 15.23 0)
+			(start 7.34 2.375)
+			(end -7.34 2.375)
 			(stroke
-				(width 0.12)
+				(width 0.127)
 				(type solid)
 			)
@@
 		)
 		(fp_line
-			(start -1.45 -2.05)
-			(end -1.45 2.05)
+			(start -7.59 -2.625)
+			(end 7.59 -2.625)
 			(stroke
 				(width 0.05)
@@
 		)
 		(fp_line
-			(start -1.45 2.05)
-			(end 21.77 2.05)
+			(start -7.59 2.625)
+			(end -7.59 -2.625)
 			(stroke
 				(width 0.05)
@@
 		)
 		(fp_line
-			(start 21.77 -2.05)
-			(end -1.45 -2.05)
+			(start 7.59 -2.625)
+			(end 7.59 2.625)
 			(stroke
 				(width 0.05)
@@
 		)
 		(fp_line
-			(start 21.77 2.05)
-			(end 21.77 -2.05)
+			(start 7.59 2.625)
+			(end -7.59 2.625)
 			(stroke
 				(width 0.05)
@@
 		)
 		(fp_line
-			(start 0 0)
-			(end 5.21 0)
-			(stroke
-				(width 0.1)
-				(type solid)
-			)
-			(layer "F.Fab")
-		)
-		(fp_line
-			(start 5.21 -1.8)
-			(end 5.21 1.8)
-			(stroke
-				(width 0.1)
-				(type solid)
-			)
-			(layer "F.Fab")
-		)
-		(fp_line
-			(start 5.21 1.8)
-			(end 15.11 1.8)
+			(start -7.34 -2.375)
+			(end 7.34 -2.375)
 			(stroke
-				(width 0.1)
+				(width 0.127)
 				(type solid)
 			)
@@
 		)
 		(fp_line
-			(start 15.11 -1.8)
-			(end 5.21 -1.8)
+			(start -7.34 2.375)
+			(end -7.34 -2.375)
 			(stroke
-				(width 0.1)
+				(width 0.127)
 				(type solid)
 			)
@@
 		)
 		(fp_line
-			(start 15.11 1.8)
-			(end 15.11 -1.8)
+			(start 7.34 -2.375)
+			(end 7.34 2.375)
 			(stroke
-				(width 0.1)
+				(width 0.127)
 				(type solid)
 			)
@@
 		)
 		(fp_line
-			(start 20.32 0)
-			(end 15.11 0)
+			(start 7.34 2.375)
+			(end -7.34 2.375)
 			(stroke
-				(width 0.1)
+				(width 0.127)
 				(type solid)
 			)
 			(layer "F.Fab")
 		)
-		(fp_text user "${REFERENCE}"
-			(at 10.16 0 0)
-			(layer "F.Fab")
-			(effects
-				(font
-					(size 1 1)
-					(thickness 0.15)
-				)
-			)
-		)
-		(pad "1" thru_hole circle
-			(at 0 0)
-			(size 2.4 2.4)
-			(drill 1.2)
+		(pad "1_1" thru_hole circle
+			(at -5.895 0)
+			(size 2.55 2.55)
+			(drill 1.7)
 			(layers "*.Cu" "*.Mask")
 			(remove_unused_layers no)
 			(net 14 "+12V")
 			(pintype "passive")
+			(solder_mask_margin 0.102)
 		)
-		(pad "2" thru_hole oval
-			(at 20.32 0)
-			(size 2.4 2.4)
-			(drill 1.2)
+		(pad "1_2" thru_hole circle
+			(at -2.235 0)
+			(size 2.55 2.55)
+			(drill 1.7)
+			(layers "*.Cu" "*.Mask")
+			(remove_unused_layers no)
+			(solder_mask_margin 0.102)
+		)
+		(pad "2_1" thru_hole circle
+			(at 2.235 0)
+			(size 2.55 2.55)
+			(drill 1.7)
 			(layers "*.Cu" "*.Mask")
 			(remove_unused_layers no)
 			(net 40 "Net-(J18-Pin_3)")
 			(pintype "passive")
+			(solder_mask_margin 0.102)
 		)
-		(embedded_fonts no)
-		(model "${KICAD9_3DMODEL_DIR}/Resistor_THT.3dshapes/R_Axial_DIN0411_L9.9mm_D3.6mm_P20.32mm_Horizontal.wrl"
-			(offset
-				(xyz 0 0 0)
-			)
-			(scale
-				(xyz 1 1 1)
-			)
-			(rotate
-				(xyz 0 0 0)
-			)
+		(pad "2_2" thru_hole circle
+			(at 5.895 0)
+			(size 2.55 2.55)
+			(drill 1.7)
+			(layers "*.Cu" "*.Mask")
+			(remove_unused_layers no)
+			(solder_mask_margin 0.102)
 		)
+		(embedded_fonts no)
 	)
 	(footprint "3544-2:FUSE_3544-2"
@@
 	)
 	(segment
-		(start 168.4613 136.652)
-		(end 168.4613 139.8947)
+		(start 171.8028 121.2088)
+		(end 180.4755 121.2088)
 		(width 4)
 		(layer "F.Cu")
@@
 	)
 	(segment
-		(start 171.8028 121.2088)
-		(end 180.4755 121.2088)
+		(start 170.7473 109.093)
+		(end 168.1819 106.5276)
 		(width 4)
 		(layer "F.Cu")
@@
 	)
 	(segment
-		(start 170.7473 109.093)
-		(end 168.1819 106.5276)
+		(start 171.09 142.24)
+		(end 171.09 139.2807)
 		(width 4)
 		(layer "F.Cu")
@@
 	)
 	(segment
-		(start 168.4613 139.8947)
-		(end 165.1 143.256)
+		(start 180.4755 121.2088)
+		(end 188.0701 113.6142)
 		(width 4)
 		(layer "F.Cu")
@@
 	)
 	(segment
-		(start 180.4755 121.2088)
-		(end 188.0701 113.6142)
+		(start 171.09 139.2807)
+		(end 168.4613 136.652)
 		(width 4)
 		(layer "F.Cu")
@@
 	)
 	(segment
-		(start 189.992 143.256)
+		(start 179.22 140.436878)
+		(end 181.042878 138.614)
+		(width 4)
+		(layer "F.Cu")
+		(net 40)
+	)
+	(segment
+		(start 179.22 142.24)
+		(end 179.22 140.436878)
+		(width 4)
+		(layer "F.Cu")
+		(net 40)
+	)
+	(segment
+		(start 188.652 138.614)
 		(end 191.643 141.605)
 		(width 4)
@@
 	)
 	(segment
-		(start 185.42 143.256)
-		(end 189.992 143.256)
+		(start 181.042878 138.614)
+		(end 188.652 138.614)
 		(width 4)
 		(layer "F.Cu")
 		(net 40)
+	)
+	(segment
+		(start 191.135 141.605)
+		(end 191.643 141.605)
+		(width 0.25)
+		(layer "F.Cu")
+		(net 40)
