File: BandPassFilter/25kHz-Band-Pass-Filter/25kHz-Band-Pass-Filter.kicad_sch (KiCad schematic)
At the start: 68 parts, among them J1 Conn_01x02, J2 Conn_01x02, J3 Conn_01x02, J4 Conn_01x02, U1 ${SIM.PARAMS}, U10 ${SIM.PARAMS}, U11 ${SIM.PARAMS}, U12 ${SIM.PARAMS}, U13 ${SIM.PARAMS}, U14 LTC2171CUKG-14_PBF, U2 ${SIM.PARAMS}, U3 ${SIM.PARAMS}, U4 MCP6S21-I_SN, U5 ${SIM.PARAMS}, U6 ${SIM.PARAMS}, U7 ${SIM.PARAMS}, U8 ${SIM.PARAMS}, U9 ${SIM.PARAMS}

Commit message: Updated capacitor/resistor values for Band Pass Filter
Parts:
- C1, C2: value 6.6nF -> 660pF
- C3, C4: value 6.1nF -> 620pF
- C7, C8: value 5.5nF -> 5.6nF
- R11, R15, R19, R23, R27, R3, R31, R7: value 100kΩ -> 6.2MΩ
Changed lines of the file:
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@@
 			)
 		)
-		(property "Value" "5.5nF"
+		(property "Value" "5.6nF"
 			(at 222.25 152.4 90)
 			(effects
@@
 			)
 		)
-		(property "Value" "100kΩ"
+		(property "Value" "6.2MΩ"
 			(at 314.96 104.1399 0)
 			(effects
@@
 			)
 		)
-		(property "Value" "100kΩ"
+		(property "Value" "6.2MΩ"
 			(at 314.96 180.3399 0)
 			(effects
@@
 			)
 		)
-		(property "Value" "6.6nF"
+		(property "Value" "660pF"
 			(at 222.25 76.2 90)
 			(effects
@@
 			)
 		)
-		(property "Value" "100kΩ"
+		(property "Value" "6.2MΩ"
 			(at 314.96 255.2699 0)
 			(effects
@@
 			)
 		)
-		(property "Value" "100kΩ"
+		(property "Value" "6.2MΩ"
 			(at 238.76 177.7999 0)
 			(effects
@@
 			)
 		)
-		(property "Value" "6.1nF"
+		(property "Value" "620pF"
 			(at 308.61 97.7899 0)
 			(effects
@@
 			)
 		)
-		(property "Value" "6.6nF"
+		(property "Value" "660pF"
 			(at 209.55 76.2 90)
 			(effects
@@
 			)
 		)
-		(property "Value" "100kΩ"
+		(property "Value" "6.2MΩ"
 			(at 238.76 101.5999 0)
 			(effects
@@
 			)
 		)
-		(property "Value" "100kΩ"
+		(property "Value" "6.2MΩ"
 			(at 238.76 252.7299 0)
 			(effects
@@
 			)
 		)
-		(property "Value" "6.1nF"
+		(property "Value" "620pF"
 			(at 304.8 69.85 90)
 			(effects
@@
 			)
 		)
-		(property "Value" "5.5nF"
+		(property "Value" "5.6nF"
 			(at 209.55 152.4 90)
 			(effects
@@
 			)
 		)
-		(property "Value" "100kΩ"
+		(property "Value" "6.2MΩ"
 			(at 240.03 328.9299 0)
 			(effects
@@
 			)
 		)
-		(property "Value" "100kΩ"
+		(property "Value" "6.2MΩ"
 			(at 316.23 331.4699 0)
 			(effects
